File: light_switch_smd2.sch (EAGLE design)
At the start: 17 parts, among them J2 SW1, T1 BT136, U1 LM1117

Commit message: v.2 Final
Changed lines of the file:
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@@
 <pinref part="LAMP" gate="G$1" pin="1"/>
 <wire x1="132.08" y1="38.1" x2="116.84" y2="38.1" width="0.1524" layer="91"/>
+<junction x="116.84" y="38.1"/>
 </segment>
 </net>

Commit message: version 3, several correction added
Parts:
- AC: value (none) -> AC
- LAMP: value (none) -> LAMP
Changed lines of the file:
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@@
 <part name="U$1" library="myblog_library" deviceset="HI-LINK5V-ACDC" device=""/>
 <part name="GND4" library="supply1" deviceset="GND" device=""/>
-<part name="LAMP" library="SparkFun-Connectors" deviceset="M03" device="1X03_NO_SILK"/>
-<part name="AC" library="SparkFun-Connectors" deviceset="M03" device="1X03_NO_SILK"/>
+<part name="LAMP" library="SparkFun-Connectors" deviceset="M03" device="1X03_NO_SILK" value="LAMP"/>
+<part name="AC" library="SparkFun-Connectors" deviceset="M03" device="1X03_NO_SILK" value="AC"/>
 </parts>
 <sheets>
